File: rocketBeaconModule_v1.1/CC1200.kicad_sch (KiCad schematic)
At the start: 36 parts, among them P1 AntMount, U3 CC1200, X1 40MHz

Commit message: backup v1.1; add part numbers
Parts:
- C15, C17, C18, C19, C23, C24, C25, C28, C29: JLCPCB# C508865 -> (none)
- C16: JLCPCB# C16772 -> (none)
- C20, C22: JLCPCB# C15195 -> (none)
- C21: JLCPCB# C152808 -> (none)
- C26: JLCPCB# C335543 -> (none)
- C27: JLCPCB# C126492 -> (none)
- C30: JLCPCB# C86288 -> (none)
- C31, C36: JLCPCB# C32949 -> (none)
- C32, C33, C35: JLCPCB# C281761 -> (none)
- C34: JLCPCB# C159806 -> (none)
- C37: JLCPCB# C325456 -> (none)
- L1, L2: JLCPCB# C76777 -> (none)
- L3, L4: JLCPCB# C12669 -> (none)
- L5, L6: JLCPCB# C27143 -> (none)
- L7: JLCPCB# C2042359 -> (none)
- L8: JLCPCB# C12670 -> (none)
- P1: JLCPCB# C504007 -> (none)
- R8: JLCPCB# C25796 -> (none)
- R9: value 18k -> 18; JLCPCB# C25084 -> (none)
- U3: JLCPCB# C122881 -> (none)
- X1: value 40MHz -> 40mhz; JLCPCB# C9010 -> (none)
Changed lines of the file:
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@@
-      (effects (font (size 1.27 1.27)) hide)
-    )
-    (property "JLCPCB#" "C122881" (id 4) (at 113.03 73.66 0)
       (effects (font (size 1.27 1.27)) hide)
     )
@@
       (effects (font (size 1.27 1.27)) hide)
     )
-    (property "JLCPCB#" "C508865" (id 4) (at 168.91 66.04 0)
-      (effects (font (size 1.27 1.27)) hide)
-    )
     (pin "1")
     (pin "2")
@@
       (effects (font (size 1.27 1.27)) hide)
     )
-    (property "JLCPCB#" "C12670" (id 4) (at 237.49 124.46 0)
-      (effects (font (size 1.27 1.27)) hide)
-    )
     (pin "1")
     (pin "2")
@@
       (effects (font (size 1.27 1.27)) hide)
     )
-    (property "JLCPCB#" "C12669" (id 4) (at 194.31 83.82 0)
-      (effects (font (size 1.27 1.27)) hide)
-    )
     (pin "1")
     (pin "2")
@@
     )
     (property "Datasheet" "https://datasheet.lcsc.com/lcsc/1811061736_Walsin-Tech-Corp-0402N100J500CT_C301961.pdf" (id 3) (at 185.42 62.23 0)
-      (effects (font (size 1.27 1.27)) hide)
-    )
-    (property "JLCPCB#" "C32949" (id 4) (at 185.42 62.23 0)
       (effects (font (size 1.27 1.27)) hide)
     )
@@
       (effects (font (size 1.27 1.27)) hide)
     )
-    (property "JLCPCB#" "C152808" (id 4) (at 139.7 77.47 0)
-      (effects (font (size 1.27 1.27)) hide)
-    )
     (pin "1")
     (pin "2")
@@
       (effects (font (size 1.27 1.27)) hide)
     )
-    (property "JLCPCB#" "C508865" (id 4) (at 148.59 69.85 0)
-      (effects (font (size 1.27 1.27)) hide)
-    )
     (pin "1")
     (pin "2")
@@
       (effects (font (size 1.27 1.27)) hide)
     )
-    (property "JLCPCB#" "C508865" (id 4) (at 64.77 99.06 0)
-      (effects (font (size 1.27 1.27)) hide)
-    )
     (pin "1")
     (pin "2")
@@
       (effects (font (size 1.27 1.27)) hide)
     )
-    (property "JLCPCB#" "C32949" (id 4) (at 209.55 62.23 0)
-      (effects (font (size 1.27 1.27)) hide)
-    )
     (pin "1")
     (pin "2")
@@
       (effects (font (size 1.27 1.27)) hide)
     )
-    (property "JLCPCB#" "C508865" (id 4) (at 149.86 85.09 0)
-      (effects (font (size 1.27 1.27)) hide)
-    )
     (pin "1")
     (pin "2")
@@
     )
     (property "Datasheet" "https://datasheet.lcsc.com/lcsc/1811081510_Murata-Electronics-GCM1555C1H101JA16D_C126492.pdf" (id 3) (at 158.75 137.16 0)
-      (effects (font (size 1.27 1.27)) hide)
-    )
-    (property "JLCPCB#" "C126492" (id 4) (at 158.75 137.16 0)
       (effects (font (size 1.27 1.27)) hide)
     )
@@
       (effects (font (size 1.27 1.27)) hide)
     )
-    (property "JLCPCB#" "C281761" (id 4) (at 193.04 73.66 0)
-      (effects (font (size 1.27 1.27)) hide)
-    )
     (pin "1")
     (pin "2")
@@
       (effects (font (size 1.27 1.27)) hide)
     )
-    (property "JLCPCB#" "C2042359" (id 4) (at 222.25 124.46 0)
-      (effects (font (size 1.27 1.27)) hide)
-    )
     (pin "1")
     (pin "2")
@@
     )
     (property "Datasheet" "https://datasheet.lcsc.com/lcsc/2206010100_UNI-ROYAL-Uniroyal-Elec-0402WGF5602TCE_C25796.pdf" (id 3) (at 90.17 113.03 0)
-      (effects (font (size 1.27 1.27)) hide)
-    )
-    (property "JLCPCB#" "C25796" (id 4) (at 90.17 113.03 0)
       (effects (font (size 1.27 1.27)) hide)
     )
@@
       (effects (font (size 1.27 1.27)) hide)
     )
-    (property "JLCPCB#" "C508865" (id 4) (at 158.75 58.42 0)
-      (effects (font (size 1.27 1.27)) hide)
-    )
     (pin "1")
     (pin "2")
@@
       (effects (font (size 1.27 1.27)) hide)
     )
-    (property "JLCPCB#" "C15195" (id 4) (at 142.24 137.16 0)
-      (effects (font (size 1.27 1.27)) hide)
-    )
     (pin "1")
     (pin "2")
@@
     )
     (property "Datasheet" "https://datasheet.lcsc.com/lcsc/2004071033_TDK-CGA2B2X7R1C473KT0Y0F_C508865.pdf" (id 3) (at 49.53 67.31 0)
-      (effects (font (size 1.27 1.27)) hide)
-    )
-    (property "JLCPCB#" "C508865" (id 4) (at 49.53 67.31 0)
       (effects (font (size 1.27 1.27)) hide)
     )
@@
       (effects (font (size 1.27 1.27)) hide)
     )
-    (property "JLCPCB#" "C508865" (id 4) (at 168.91 76.2 0)
-      (effects (font (size 1.27 1.27)) hide)
-    )
     (pin "1")
     (pin "2")
@@
       (effects (font (size 1.27 1.27)) hide)
     )
-    (property "JLCPCB#" "C12669" (id 4) (at 194.31 106.68 0)
-      (effects (font (size 1.27 1.27)) hide)
-    )
     (pin "1")
     (pin "2")
@@
       (effects (font (size 1.27 1.27)) hide)
     )
-    (property "JLCPCB#" "C159806" (id 4) (at 195.58 134.62 0)
-      (effects (font (size 1.27 1.27)) hide)
-    )
     (pin "1")
     (pin "2")
@@
     )
     (property "Datasheet" "https://datasheet.lcsc.com/lcsc/2004071033_TDK-CGA2B2X7R1C473KT0Y0F_C508865.pdf" (id 3) (at 67.31 52.07 0)
-      (effects (font (size 1.27 1.27)) hide)
-    )
-    (property "JLCPCB#" "C508865" (id 4) (at 67.31 52.07 0)
       (effects (font (size 1.27 1.27)) hide)
     )
@@
       (effects (font (size 1.27 1.27)) hide)
     )
-    (property "JLCPCB#" "C281761" (id 4) (at 194.31 96.52 0)
-      (effects (font (size 1.27 1.27)) hide)
-    )
     (pin "1")
     (pin "2")
@@
       (effects (font (size 1.27 1.27)) hide)
     )
-    (property "JLCPCB#" "C76777" (id 4) (at 142.24 111.76 0)
-      (effects (font (size 1.27 1.27)) hide)
-    )
     (pin "1")
     (pin "2")
@@
       (effects (font (size 1.27 1.27)) hide)
     )
-    (property "JLCPCB#" "C27143" (id 4) (at 208.28 106.68 0)
-      (effects (font (size 1.27 1.27)) hide)
-    )
     (pin "1")
     (pin "2")
@@
     (in_bom yes) (on_board yes)
     (property "Reference" "X1" (id 0) (at 203.2 53.34 0))
-    (property "Value" "40MHz" (id 1) (at 205.74 55.88 0))
+    (property "Value" "40mhz" (id 1) (at 205.74 55.88 0))
     (property "Footprint" "Oscillator:Oscillator_SMD_Abracon_ASE-4Pin_3.2x2.5mm" (id 2) (at 199.39 58.42 0)
       (effects (font (size 1.27 1.27)) hide)
     )
     (property "Datasheet" "https://abracon.com/Resonators/ABM8W.pdf" (id 3) (at 199.39 58.42 0)
-      (effects (font (size 1.27 1.27)) hide)
-    )
-    (property "JLCPCB#" "C9010" (id 4) (at 199.39 58.42 0)
       (effects (font (size 1.27 1.27)) hide)
     )
@@
       (effects (font (size 1.27 1.27)) (justify left))
     )
-    (property "Value" "18k" (id 1) (at 143.51 127 0)
+    (property "Value" "18" (id 1) (at 143.51 127 0)
       (effects (font (size 1.27 1.27)) (justify left))
     )
@@
       (effects (font (size 1.27 1.27)) hide)
     )
-    (property "JLCPCB#" "C25084" (id 4) (at 142.24 125.73 0)
-      (effects (font (size 1.27 1.27)) hide)
-    )
     (pin "1")
     (pin "2")
@@
     )
     (property "Datasheet" "https://jlcpcb.com/partdetail/Tdk-CGA2B2X7R1C473KT0Y0F/C508865" (id 3) (at 64.77 69.85 0)
-      (effects (font (size 1.27 1.27)) hide)
-    )
-    (property "JLCPCB#" "C16772" (id 4) (at 64.77 69.85 0)
       (effects (font (size 1.27 1.27)) hide)
     )
@@
       (effects (font (size 1.27 1.27)) hide)
     )
-    (property "JLCPCB#" "C15195" (id 4) (at 137.16 88.9 0)
-      (effects (font (size 1.27 1.27)) hide)
-    )
     (pin "1")
     (pin "2")
@@
       (effects (font (size 1.27 1.27)) hide)
     )
-    (property "JLCPCB#" "C325456" (id 4) (at 229.87 132.08 0)
-      (effects (font (size 1.27 1.27)) hide)
-    )
     (pin "1")
     (pin "2")
@@
     )
     (property "Datasheet" "https://datasheet.lcsc.com/lcsc/1810241229_YAGEO-CC0402CRNPO9BN5R1_C281761.pdf" (id 3) (at 208.28 118.11 0)
-      (effects (font (size 1.27 1.27)) hide)
-    )
-    (property "JLCPCB#" "C281761" (id 4) (at 208.28 118.11 0)
       (effects (font (size 1.27 1.27)) hide)
     )
@@
     )
     (property "Datasheet" "https://datasheet.lcsc.com/lcsc/1811081511_Murata-Electronics-LQG15HS56NJ02D_C162544.pdf" (id 3) (at 180.34 90.17 0)
-      (effects (font (size 1.27 1.27)) hide)
-    )
-    (property "JLCPCB#" "C76777" (id 4) (at 180.34 90.17 0)
       (effects (font (size 1.27 1.27)) hide)
     )
@@
       (effects (font (size 1.27 1.27)) hide)
     )
-    (property "JLCPCB#" "C27143" (id 4) (at 195.58 124.46 0)
-      (effects (font (size 1.27 1.27)) hide)
-    )
     (pin "1")
     (pin "2")
@@
       (effects (font (size 1.27 1.27)) hide)
     )
-    (property "JLCPCB#" "C86288" (id 4) (at 175.26 124.46 0)
-      (effects (font (size 1.27 1.27)) hide)
-    )
     (pin "1")
     (pin "2")
@@
       (effects (font (size 1.27 1.27)) hide)
     )
-    (property "JLCPCB#" "C335543" (id 4) (at 158.75 125.73 0)
-      (effects (font (size 1.27 1.27)) hide)
-    )
     (pin "1")
     (pin "2")
@@
     )
     (property "Datasheet" "https://datasheet.lcsc.com/lcsc/2004071033_TDK-CGA2B2X7R1C473KT0Y0F_C508865.pdf" (id 3) (at 76.2 107.95 0)
-      (effects (font (size 1.27 1.27)) hide)
-    )
-    (property "JLCPCB#" "C508865" (id 4) (at 76.2 107.95 0)
       (effects (font (size 1.27 1.27)) hide)
     )
@@
       (effects (font (size 1.27 1.27)) hide)
     )
-    (property "JLCPCB#" "C504007" (id 4) (at 254 124.46 0)
-      (effects (font (size 1.27 1.27)) hide)
-    )
