File: rocketBeaconModule_v1.1/rocketBeaconModule.kicad_sch (KiCad schematic)
At the start: 36 parts, among them J1 TYPE-C-31-M-12, J2 Jumper Select, J3 Main Bus, U1 STM32F401CCU6, U2 AMS1117-3.3, Y1 16MHz

Commit message: backup v1.1; add part numbers
Parts:
- C1, C4, C5, C7, C8: value 100nF -> 100n; JLCPCB# C307331 -> (none)
- C10: value 10nF -> 10n; JLCPCB# C15195 -> (none)
- C11, C12: value 1uF -> 1u; JLCPCB# C52923 -> (none)
- C13, C14: value 22uF -> 22u; JLCPCB# C5674 -> (none)
- C2: value 10uF -> 10u; JLCPCB# C19702 -> (none)
- C3, C6: value 10pF -> 10p; JLCPCB# C32949 -> (none)
- C9: value 2.2uF -> 2.2u; JLCPCB# C12530 -> (none)
- D1: JLCPCB# C273598 -> (none)
- D2: JLCPCB# C273602 -> (none)
- D3: JLCPCB# C273603 -> (none)
- FB1: JLCPCB# C85831 -> (none)
- J1: JLCPCB# C165948 -> (none)
- J2, SWD1: JLCPCB# C124378 -> (none)
- J3: JLCPCB# C124418 -> (none)
- R1, R2: JLCPCB# C25867 -> (none)
- R3, R4: JLCPCB# C25906 -> (none)
- R5, R6, R7: JLCPCB# C11702 -> (none)
- U1: JLCPCB# C79861 -> (none)
- U2: JLCPCB# C6186 -> (none)
- Y1: JLCPCB# C13738 -> (none)
